File: electronics/v1/ws.sch (KiCad schematic (older format))
At the start: 33 parts, among them J1 PWR, J2 Recevier, Q1 TN0604G, Q2 TP0610L, SW1 SW_Push, U1 WeMos_D1_mini, U2 L7805, U3 EA-DOGM128W-6, U4 BME280_I2C_Board

Commit message: schematic update
Parts:
- removed C3: .1uF, Capacitor_THT:C_Rect_L7.0mm_W2.0mm_P5.00mm, symbol Device:C
- removed Q2: TP0610L, Package_TO_SOT_THT:TO-92L_Inline, symbol Transistor_FET:TP0610L
- removed R3, R8: 10K, Resistor_THT:R_Axial_DIN0207_L6.3mm_D2.5mm_P10.16mm_Horizontal, symbol Device:R
- removed U2: L7805, Package_TO_SOT_THT:TO-220-3_Vertical, symbol Regulator_Linear:L7805
- added C3: 2.2uF, Capacitor_THT:CP_Radial_D5.0mm_L10mm_P2.50mm_Lying, symbol Device:CP
- added U2: LF50_TO220, Package_TO_SOT_THT:TO-220-3_Horizontal_TabDown, symbol Regulator_Linear:LF50_TO220
- C1: value .33uF -> .1uF
- R1: value 100R -> 47k
- R2: value 10K -> 65k
- R7: renamed from R9; value 60R -> 220R
- R8: renamed from R10; value 60R -> 220R
- R9: renamed from R11; value 60R -> 220R
- renumbered R4 to R3, R5 to R4, R6 to R5, R7 to R6
Connections:
- net labels added: D6
- net labels removed: D4
- wire segments 93 -> 84
Other:
- moved on the sheet: Q1, R6

Commit message: got radio working; verified backlight
Parts:
- R7, R8, R9: value 220R -> 100R
Connections:
- wire segments 84 -> 83
Changed lines of the file:
@@
 TX
-Wire Wire Line
-	7250 2250 7250 2350
 Wire Wire Line
 	9700 1450 9850 1450
@@
 P 8450 1750
 F 0 "R9" V 8550 1800 50  0000 C CNN
-F 1 "220R" V 8350 1800 50  0000 C CNN
+F 1 "100R" V 8350 1800 50  0000 C CNN
 F 2 "Resistor_THT:R_Axial_DIN0207_L6.3mm_D2.5mm_P10.16mm_Horizontal" V 8380 1750 50  0001 C CNN
 F 3 "~" H 8450 1750 50  0001 C CNN
@@
 P 8450 1450
 F 0 "R8" V 8550 1500 50  0000 C CNN
-F 1 "220R" V 8350 1500 50  0000 C CNN
+F 1 "100R" V 8350 1500 50  0000 C CNN
 F 2 "Resistor_THT:R_Axial_DIN0207_L6.3mm_D2.5mm_P10.16mm_Horizontal" V 8380 1450 50  0001 C CNN
 F 3 "~" H 8450 1450 50  0001 C CNN
@@
 P 8450 1150
 F 0 "R7" V 8550 1200 50  0000 C CNN
-F 1 "220R" V 8350 1200 50  0000 C CNN
+F 1 "100R" V 8350 1200 50  0000 C CNN
 F 2 "Resistor_THT:R_Axial_DIN0207_L6.3mm_D2.5mm_P10.16mm_Horizontal" V 8380 1150 50  0001 C CNN
 F 3 "~" H 8450 1150 50  0001 C CNN

Commit message: designed PCB
Parts:
- removed R3: 10k, Resistor_THT:R_Axial_DIN0207_L6.3mm_D2.5mm_P10.16mm_Horizontal, symbol Device:R
- removed SC1: Solar_Cell, Connector_PinHeader_2.54mm:PinHeader_1x02_P2.54mm_Vertical, symbol Device:Solar_Cell
- added R3: GL5516, OptoDevice:R_LDR_5.1x4.3mm_P3.4mm_Vertical, symbol Device:R_PHOTO
- C2: footprint Capacitor_THT:CP_Radial_D10.0mm_P5.00mm -> CustomParts:CP_Radial_D10.0mm_L18mm_P5.0mm_Lying
- R4: value 10k -> 5k
Connections:
- wire segments 83 -> 80
Other:
- moved on the sheet: R4
Changed lines of the file:
@@
 F 0 "C2" H 1718 1796 50  0000 L CNN
 F 1 "1000uF" H 1718 1705 50  0000 L CNN
-F 2 "Capacitor_THT:CP_Radial_D10.0mm_P5.00mm" H 1638 1600 50  0001 C CNN
+F 2 "CustomParts:CP_Radial_D10.0mm_L18mm_P5.0mm_Lying" H 1638 1600 50  0001 C CNN
 F 3 "~" H 1600 1750 50  0001 C CNN
 	1    1600 1750
@@
 	1    0    0    -1
 $EndComp
-$Comp
-L Device:Solar_Cell SC1
-U 1 1 62F0A31C
-P 4450 1550
-F 0 "SC1" H 4282 1646 50  0000 R CNN
-F 1 "Solar_Cell" H 4282 1555 50  0000 R CNN
-F 2 "Connector_PinHeader_2.54mm:PinHeader_1x02_P2.54mm_Vertical" V 4450 1610 50  0001 C CNN
-F 3 "~" V 4450 1610 50  0001 C CNN
-	1    4450 1550
-	-1   0    0    -1
-$EndComp
 Text GLabel 3900 1800 0    50   Input ~ 0
 GND
@@
 A0
 $Comp
-L Device:R R3
-U 1 1 62F1F5D9
-P 4150 1350
-F 0 "R3" H 4220 1396 50  0000 L CNN
-F 1 "10k" H 4220 1305 50  0000 L CNN
-F 2 "Resistor_THT:R_Axial_DIN0207_L6.3mm_D2.5mm_P10.16mm_Horizontal" V 4080 1350 50  0001 C CNN
-F 3 "~" H 4150 1350 50  0001 C CNN
-	1    4150 1350
-	-1   0    0    -1
-$EndComp
-$Comp
 L Device:R R4
 U 1 1 62F2A697
-P 4150 1650
-F 0 "R4" H 4220 1696 50  0000 L CNN
-F 1 "10k" H 4220 1605 50  0000 L CNN
-F 2 "Resistor_THT:R_Axial_DIN0207_L6.3mm_D2.5mm_P10.16mm_Horizontal" V 4080 1650 50  0001 C CNN
-F 3 "~" H 4150 1650 50  0001 C CNN
-	1    4150 1650
-	-1   0    0    -1
-$EndComp
-Wire Wire Line
-	3900 1500 4150 1500
-Connection ~ 4150 1500
-Wire Wire Line
-	4150 1200 4450 1200
-Wire Wire Line
-	4450 1200 4450 1350
-Wire Wire Line
-	3900 1800 4150 1800
-Wire Wire Line
-	4150 1800 4450 1800
-Wire Wire Line
-	4450 1800 4450 1650
-Connection ~ 4150 1800
+P 4400 1650
+F 0 "R4" H 4470 1696 50  0000 L CNN
+F 1 "5k" H 4470 1605 50  0000 L CNN
+F 2 "Resistor_THT:R_Axial_DIN0207_L6.3mm_D2.5mm_P10.16mm_Horizontal" V 4330 1650 50  0001 C CNN
+F 3 "~" H 4400 1650 50  0001 C CNN
+	1    4400 1650
+	-1   0    0    -1
+$EndComp
 Text GLabel 1600 3350 2    50   Input ~ 0
 A0
@@
 Wire Wire Line
 	2850 2700 2850 3150
+$Comp
+L Device:R_PHOTO R3
+U 1 1 62F6C18F
+P 4400 1350
+F 0 "R3" H 4600 1400 50  0000 R CNN
+F 1 "GL5516" H 4750 1300 50  0000 R CNN
+F 2 "OptoDevice:R_LDR_5.1x4.3mm_P3.4mm_Vertical" V 4450 1100 50  0001 L CNN
+F 3 "~" H 4400 1300 50  0001 C CNN
+	1    4400 1350
+	-1   0    0    -1
+$EndComp
+Connection ~ 4400 1500
+Text GLabel 3900 1200 0    50   Input ~ 0
+3V3
+Wire Wire Line
+	3900 1200 4400 1200
+Wire Wire Line
+	3900 1500 4400 1500
+Wire Wire Line
+	3900 1800 4400 1800
 $EndSCHEMATC

Commit message: schematic correction (R4 exact value)
Parts:
- R4: value 5k -> 5.1k
Changed lines of the file:
@@
 P 4400 1650
 F 0 "R4" H 4470 1696 50  0000 L CNN
-F 1 "5k" H 4470 1605 50  0000 L CNN
+F 1 "5.1k" H 4470 1605 50  0000 L CNN
 F 2 "Resistor_THT:R_Axial_DIN0207_L6.3mm_D2.5mm_P10.16mm_Horizontal" V 4330 1650 50  0001 C CNN
 F 3 "~" H 4400 1650 50  0001 C CNN
