File: electronics/outdoor-v2/outdoor.kicad_pcb (KiCad board)
At the start: 2 copper layers, 60 x 30 mm, 9 parts, among them J1 TX433MHz, U1 ATtiny85V-10PU, U2 DS18B20

Commit message: outdoor unit revision WIP
Parts:
- removed D1: 1N60, Diode_THT:D_DO-35_SOD27_P10.16mm_Horizontal
- removed D2: 4.3V, Diode_THT:D_DO-35_SOD27_P10.16mm_Horizontal
- removed SC1: 5V, Connector_PinHeader_2.54mm:PinHeader_1x02_P2.54mm_Vertical
- added C1: 1u, Capacitor_THT:C_Rect_L7.0mm_W2.5mm_P5.00mm, F.Cu at (57.1, 83.2)
- added C2: 1u, Capacitor_THT:C_Rect_L7.0mm_W2.5mm_P5.00mm, F.Cu at (47.0, 83.0)
- added R3: 10k, Resistor_THT:R_Axial_DIN0207_L6.3mm_D2.5mm_P10.16mm_Horizontal, F.Cu at (72.6, 91.2)
- added R4: 4.7k, Resistor_THT:R_Axial_DIN0207_L6.3mm_D2.5mm_P10.16mm_Horizontal, F.Cu at (56.0, 92.7)
- added SW1: SW_Push, Button_Switch_THT:SW_PUSH_6mm, F.Cu at (45.5, 92.2)
- added U3: DS18B20, Package_TO_SOT_THT:TO-92_Inline_Wide, F.Cu at (88.5, 161.5)
- BT1: value 3xNiCd -> 4.5V; footprint CustomParts:NiCd-Small -> Connector_PinHeader_2.54mm:PinHeader_1x02_P2.54mm_Vertical
- R1: value 59 -> 1M
- R2: value 4.7k -> 100k
- U1: value ATtiny85V-10PU -> MCP1700-3302E; footprint Package_DIP:DIP-8_W7.62mm -> Package_TO_SOT_THT:TO-92_Inline_Wide
- U2: value DS18B20 -> ATtiny45V-10PU; footprint Package_TO_SOT_THT:TO-92_Inline_Wide -> Package_DIP:DIP-8_W7.62mm
- moved R2 26.3 mm to (72.3, 87.0), turned to 180 degrees
- moved U1 22.5 mm to (52.0, 88.0), turned to 90 degrees
- moved U2 18.4 mm to (61.0, 93.0)
- moved BT1 4.33 mm to (47.8, 101.9)
- moved R1 3.53 mm to (62.1, 83.0), turned to 0 degrees
- moved J1 0.46 mm to (84.2, 103.1)
Connections:
- J1 pad 2: Net-(J1-Pad2) -> Net-(BT1-Pad1)
- R1 pad 1: Net-(R1-Pad1) -> Net-(BT1-Pad1)
- R1 pad 2: Net-(D1-Pad2) -> Net-(R1-Pad2)
- R2 pad 1: Net-(BT1-Pad1) -> Net-(R1-Pad2)
- R2 pad 2: Net-(R2-Pad2) -> Net-(BT1-Pad2)
- U1 pad 1: Net-(U1-Pad1) -> Net-(BT1-Pad2)
- U1 pad 2: Net-(J1-Pad2) -> Net-(BT1-Pad1)
- U1 pad 3: Net-(U1-Pad3) -> Net-(C2-Pad1)
- U2 pad 1: Net-(BT1-Pad2) -> Net-(SW1-Pad2)
- U2 pad 2: Net-(R2-Pad2) -> Net-(R1-Pad2)
- U2 pad 3: Net-(BT1-Pad1) -> (no net)
Routing:
- net Net-(C2-Pad1): track 0.00 -> 124.1 mm
- net Net-(R4-Pad2): track 0.00 -> 85.8 mm
- net Net-(BT1-Pad2): track 95.6 -> 136.5 mm
- net Net-(J1-Pad2): track 22.9 -> 0.00 mm
- net Net-(BT1-Pad1): track 49.5 -> 68.7 mm
- net Net-(R1-Pad2): track 0.00 -> 18.9 mm
- net Net-(R2-Pad2): track 17.1 -> 0.00 mm
- net Net-(SW1-Pad2): track 0.00 -> 17.0 mm
- net Net-(J1-Pad1): track 17.9 -> 27.9 mm
- net Net-(R1-Pad1): track 5.60 -> 0.00 mm
- net Net-(D1-Pad2): track 4.00 -> 0.00 mm
Other:
- board size 60 x 30 mm -> 60 x 90 mm
- board text added: "+ -"
- board text added: "Battery 3 x AAA"
- board text added: "DS18B20"
- board text added: "YAWS"
- board text added: "outdoor sensor"
- board text removed: "+5V"
- board text removed: "-"
- board text removed: "NiCd 3 cells"
